Commit message: added gazebo simulation

File: kuka_kr5_description/urdf/kr5_arc.gazebo.xacro (robot description, xacro)
@@ -18,8 +18,8 @@
     <type>transmission_interface/SimpleTransmission</type>
     <joint name="joint_a1">
-       <hardwareInterface>EffortJointInterface</hardwareInterface>
+       <hardwareInterface>hardware_interface/EffortJointInterface</hardwareInterface>
     </joint>
     <actuator name="joint_a1_actuator">
-       <hardwareInterface>hardwareInterface/EffortJointInterface</hardwareInterface>
+       <hardwareInterface>hardware_interface/EffortJointInterface</hardwareInterface>
        <mechanicalReduction>1</mechanicalReduction>
     </actuator>
@@ -28,8 +28,8 @@
    <type>transmission_interface/SimpleTransmission</type>
    <joint name="joint_a2">
-      <hardwareInterface>EffortJointInterface</hardwareInterface>
+      <hardwareInterface>hardware_interface/EffortJointInterface</hardwareInterface>
    </joint>
    <actuator name="joint_a2_actuator">
-      <hardwareInterface>EffortJointInterface</hardwareInterface>
+      <hardwareInterface>hardware_interface/EffortJointInterface</hardwareInterface>
       <mechanicalReduction>1</mechanicalReduction>
    </actuator>
@@ -38,8 +38,8 @@
    <type>transmission_interface/SimpleTransmission</type>
    <joint name="joint_a3">
-      <hardwareInterface>EffortJointInterface</hardwareInterface>
+      <hardwareInterface>hardware_interface/EffortJointInterface</hardwareInterface>
    </joint>
    <actuator name="joint_a3_actuator">
-      <hardwareInterface>EffortJointInterface</hardwareInterface>
+      <hardwareInterface>hardware_interface/EffortJointInterface</hardwareInterface>
       <mechanicalReduction>1</mechanicalReduction>
    </actuator>

File: kuka_kr5_description/urdf/kr5_arc.urdf.xacro (robot description, xacro)
@@ -303,6 +303,6 @@
     <joint name="${prefix}base_link-base" type="fixed">
       <origin xyz="0 0 0" rpy="0 0 0" />
-      <parent link="${prefix}base_link" />
-      <child link="${prefix}footprint" />
+      <parent link="${prefix}footprint" />
+      <child link="${prefix}base_link" />
     </joint>
   </xacro:macro>
