Commit message: cleanup - no more trembling etc. position controller works nicely

File: kr5_description/urdf/common.gazebo.xacro (robot description, xacro)
@@ -1,15 +1,28 @@
 <?xml version="1.0"?>
 <robot xmlns:xacro="http://ros.org/wiki/xacro">
+  <xacro:arg name="use_ros_control" default="False" />
+  <xacro:arg name="control_period" default="0.001" />
+  <xacro:arg name="motors_controller_type" default="PositionJointInterface" /> <!-- PositionJointInterface VelocityJointInterface  EffortJointInterface-->
+  <xacro:arg name="use_the_plate" default="True" />
   <gazebo>
-    <plugin name="ros_control" filename="libgazebo_ros_control.so">
-    </plugin>
-<!-- controllers: -->
-   <!--Plugin loads hardware interfaces and controller manager
-   <plugin name="gazebo_ros_control" filename="libgazebo_ros_control.so">
-      <robotNamespace>/$(arg robot_name)/joints</robotNamespace>
-      <robotSimType>gazebo_ros_control/DefaultRobotHWSim</robotSimType>
-      <controlPeriod>0.001</controlPeriod>
+    <xacro:unless value="$(arg use_ros_control)">
+      <plugin name="ros_control" filename="libgazebo_ros_control.so">
+      </plugin>
+    </xacro:unless>
+  <xacro:if value="$(arg use_ros_control)">
+  <plugin name="gazebo_ros_control" filename="libgazebo_ros_control.so">
+     <robotNamespace>/$(arg robot_name)</robotNamespace>
+     <robotSimType>gazebo_ros_control/DefaultRobotHWSim</robotSimType>
+     <controlPeriod>$(arg control_period)</controlPeriod>
+  </plugin>
+<!--<gazebo>
+   <plugin name="ground_truth" filename="libgazebo_ros_p3d.so">
+      <frameName>world</frameName>
+      <bodyName>base_link</bodyName>
+      <topicName>/gazebo/$(arg robot_name)/odom</topicName>
+      <updateRate>100.0</updateRate>
    </plugin>
--->
+</gazebo>-->
+  </xacro:if>
 <!--
     <plugin name="gazebo_ros_power_monitor_controller" filename="libgazebo_ros_power_monitor.so">

File: kr5_description/urdf/kr.gazebo.xacro (robot description, xacro)
@@ -2,29 +2,78 @@
 <robot xmlns:xacro="http://ros.org/wiki/xacro">
   <xacro:macro name="kr_arm_gazebo" params="prefix">
-    <!-- Just color the links: -->
-<gazebo reference="link_1">
-   <material>Gazebo/Green</material>
-</gazebo>
-<gazebo reference="link_2">
-   <material>Gazebo/Orange</material>
-</gazebo>
-<gazebo reference="link_3">
-   <material>Gazebo/Blue</material>
-</gazebo>
-<gazebo reference="link_4">
-   <material>Gazebo/Red</material>
-</gazebo>
-<gazebo reference="link_5">
-   <material>Gazebo/Purple</material>
-</gazebo>
-<gazebo reference="link_6">
-   <material>Gazebo/Yellow</material>
-</gazebo>
-<gazebo reference="base_link">
-   <material>Gazebo/Turquoise</material>
-</gazebo>
-<gazebo reference="ee_link">
-   <material>Gazebo/White</material>
-</gazebo>
+    <xacro:unless value="$(arg use_ros_control)">
+        <!-- Just color the links: -->
+      <gazebo reference="link_1">
+         <material>Gazebo/Green</material>
+      </gazebo>
+      <gazebo reference="link_2">
+         <material>Gazebo/Orange</material>
+      </gazebo>
+      <gazebo reference="link_3">
+         <material>Gazebo/Blue</material>
+      </gazebo>
+      <gazebo reference="link_4">
+         <material>Gazebo/Red</material>
+      </gazebo>
+      <gazebo reference="link_5">
+         <material>Gazebo/Purple</material>
+      </gazebo>
+      <gazebo reference="link_6">
+         <material>Gazebo/Yellow</material>
+      </gazebo>
+      <gazebo reference="base_link">
+         <material>Gazebo/Turquoise</material>
+      </gazebo>
+      <gazebo reference="ee_link">
+         <material>Gazebo/White</material>
+      </gazebo>
+    </xacro:unless>
+    <xacro:if value="$(arg use_ros_control)">
+      <gazebo reference="link_1">
+      <mu1>1</mu1>
+      <mu2>1</mu2>
+      <selfCollide>true</selfCollide>
+         <material>Gazebo/Green</material>
+      </gazebo>
+      <gazebo reference="link_2">
+      <mu1>1</mu1>
+      <mu2>1</mu2>
+      <selfCollide>true</selfCollide>
+         <material>Gazebo/Orange</material>
+      </gazebo>
+      <gazebo reference="link_3">
+      <mu1>1</mu1>
+      <mu2>1</mu2>
+      <selfCollide>true</selfCollide>
+         <material>Gazebo/Blue</material>
+      </gazebo>
+      <gazebo reference="link_4">
+      <mu1>1</mu1>
+      <mu2>1</mu2>
+      <selfCollide>true</selfCollide>
+         <material>Gazebo/Red</material>
+      </gazebo>
+      <gazebo reference="link_5">
+      <mu1>1</mu1>
+      <mu2>1</mu2>
+      <selfCollide>true</selfCollide>
+         <material>Gazebo/Purple</material>
+      </gazebo>
+      <gazebo reference="link_6">
+      <mu1>1</mu1>
+      <mu2>1</mu2>
+      <selfCollide>true</selfCollide>
+         <material>Gazebo/Yellow</material>
+      </gazebo>
+      <gazebo reference="base_link">
+      <mu1>1</mu1>
+      <mu2>1</mu2>
+      <selfCollide>true</selfCollide>
+         <material>Gazebo/Turquoise</material>
+      </gazebo>
+      <gazebo reference="ee_link">
+         <material>Gazebo/White</material>
+      </gazebo>
+    </xacro:if>
 <!-- p3d plugin (3D Position Interface for Ground Truth)
      This is required only for rviz that the balllink tf is known!

File: kr5_description/urdf/kr.transmission.xacro (robot description, xacro)
@@ -5,8 +5,8 @@
       <type>transmission_interface/SimpleTransmission</type>
       <joint name="${prefix}joint_a1">
-        <hardwareInterface>hardware_interface/PositionJointInterface</hardwareInterface>
+        <hardwareInterface>hardware_interface/$(arg motors_controller_type)</hardwareInterface>
       </joint>
       <actuator name="${prefix}shoulder_pan_motor">
-                  <hardwareInterface>hardware_interface/PositionJointInterface</hardwareInterface>
+        <hardwareInterface>hardware_interface/$(arg motors_controller_type)</hardwareInterface>
         <mechanicalReduction>1</mechanicalReduction>
       </actuator>
@@ -15,8 +15,8 @@
       <type>transmission_interface/SimpleTransmission</type>
       <joint name="${prefix}joint_a2">
-        <hardwareInterface>hardware_interface/PositionJointInterface</hardwareInterface>
+        <hardwareInterface>hardware_interface/$(arg motors_controller_type)</hardwareInterface>
       </joint>
       <actuator name="${prefix}shoulder_lift_motor">
-                  <hardwareInterface>hardware_interface/PositionJointInterface</hardwareInterface>
+        <hardwareInterface>hardware_interface/$(arg motors_controller_type)</hardwareInterface>
         <mechanicalReduction>1</mechanicalReduction>
       </actuator>
@@ -25,8 +25,8 @@
       <type>transmission_interface/SimpleTransmission</type>
       <joint name="${prefix}joint_a3">
-        <hardwareInterface>hardware_interface/PositionJointInterface</hardwareInterface>
+        <hardwareInterface>hardware_interface/$(arg motors_controller_type)</hardwareInterface>
       </joint>
       <actuator name="${prefix}elbow_motor">
-                  <hardwareInterface>hardware_interface/PositionJointInterface</hardwareInterface>
+        <hardwareInterface>hardware_interface/$(arg motors_controller_type)</hardwareInterface>
         <mechanicalReduction>1</mechanicalReduction>
       </actuator>
@@ -35,8 +35,8 @@
       <type>transmission_interface/SimpleTransmission</type>
       <joint name="${prefix}joint_a4">
-        <hardwareInterface>hardware_interface/PositionJointInterface</hardwareInterface>
+        <hardwareInterface>hardware_interface/$(arg motors_controller_type)</hardwareInterface>
       </joint>
       <actuator name="${prefix}wrist_1_motor">
-      <hardwareInterface>hardware_interface/PositionJointInterface</hardwareInterface>
+        <hardwareInterface>hardware_interface/$(arg motors_controller_type)</hardwareInterface>
         <mechanicalReduction>1</mechanicalReduction>
       </actuator>
@@ -45,8 +45,8 @@
       <type>transmission_interface/SimpleTransmission</type>
       <joint name="${prefix}joint_a5">
-        <hardwareInterface>hardware_interface/PositionJointInterface</hardwareInterface>
+        <hardwareInterface>hardware_interface/$(arg motors_controller_type)</hardwareInterface>
       </joint>
       <actuator name="${prefix}wrist_2_motor">
-                  <hardwareInterface>hardware_interface/PositionJointInterface</hardwareInterface>
+        <hardwareInterface>hardware_interface/$(arg motors_controller_type)</hardwareInterface>
         <mechanicalReduction>1</mechanicalReduction>
       </actuator>
@@ -55,8 +55,8 @@
       <type>transmission_interface/SimpleTransmission</type>
       <joint name="${prefix}joint_a6">
-        <hardwareInterface>hardware_interface/PositionJointInterface</hardwareInterface>
+        <hardwareInterface>hardware_interface/$(arg motors_controller_type)</hardwareInterface>
       </joint>
       <actuator name="${prefix}wrist_3_motor">
-            <hardwareInterface>hardware_interface/PositionJointInterface</hardwareInterface>
+        <hardwareInterface>hardware_interface/$(arg motors_controller_type)</hardwareInterface>
         <mechanicalReduction>1</mechanicalReduction>
       </actuator>

File: kr5_description/urdf/kr5.urdf.xacro (robot description, xacro)
@@ -4,17 +4,7 @@
        xmlns:sensor="http://playerstage.sourceforge.net/gazebo/xmlschema/#sensor"
        xmlns:xacro="http://ros.org/wiki/xacro">
-  <!-- currently not used within moveit -->
-  <xacro:arg name="motors_controller_type" default="PositionJointInterface" /> <!-- PositionJointInterface VelocityJointInterface  EffortJointInterface-->
-  <xacro:arg name="control_period" default="0.001" />
-  <xacro:arg name="use_the_plate" default="True" />
   <xacro:include filename="$(find kr5_description)/urdf/kr.transmission.xacro" />
   <xacro:include filename="$(find kr5_description)/urdf/kr.gazebo.xacro" />
   <!-- effort values can be found here: https://github.com/ros-industrial/universal_robot/issues/32-->
-  <xacro:property name="joint_effort_limit_1" value="150" />
-  <xacro:property name="joint_effort_limit_2" value="150" />
-  <xacro:property name="joint_effort_limit_3" value="150" />
-  <xacro:property name="joint_effort_limit_4" value="28" />
-  <xacro:property name="joint_effort_limit_5" value="1" />
-  <xacro:property name="joint_effort_limit_6" value="2" /><!-- let this value low! -->
   <!-- plate Properties -->
   <xacro:property name="plate_mass" value="0.5" />
@@ -182,5 +172,5 @@
            <origin xyz="0 0 0" rpy="0 0 0" />
            <geometry>
-              <mesh filename="package://kuka_manipulator_description/meshes/tools/collision/plate_40.stl" scale="0.01 0.01 0.01" /> <!-- plate is 20x20x1 m -->
+              <mesh filename="package://kr5_description/meshes/tools/plate_40.stl" scale="0.01 0.01 0.01" /> <!-- plate is 20x20x1 m -->
            </geometry>
         </visual>
@@ -188,5 +178,5 @@
            <origin xyz="0 0 0" rpy="0 0 0" />
            <geometry>
-              <mesh filename="package://kuka_manipulator_description/meshes/tools/collision/plate_40.stl" scale="0.01 0.01 0.01" />
+              <mesh filename="package://kr5_description/meshes/tools/plate_40.stl" scale="0.01 0.01 0.01" /> <!-- plate is 20x20x1 m -->
            </geometry>
         </collision>

File: kr5_description/urdf/kr5_robot.urdf.xacro (robot description, xacro)
@@ -2,9 +2,9 @@
 <robot xmlns:xacro="http://ros.org/wiki/xacro"
        name="$(arg robot_name)">>
-  <!-- common stuff -->
+  <!-- common stuff // load kr_arm_gazebo macro -->
   <xacro:include filename="$(find kr5_description)/urdf/common.gazebo.xacro" />
-  <!-- ur5 -->
+  <!-- load kr5_robot macro  -->
   <xacro:include filename="$(find kr5_description)/urdf/kr5.urdf.xacro" />
-  <!-- arm -->
+  <!-- execute macro -->
   <xacro:kr5_robot prefix=""/>
   <link name="world" />
