Commit message: added top state and haltemoment

File: ball_description/urdf/ball.gazebo.xacro (robot description, xacro)
@@ -5,11 +5,11 @@
       <maxVel>1000</maxVel>
       <minDepth>0</minDepth>
-      <mu1>0.25</mu1>
-      <mu2>0.25</mu2>
+      <mu1>10</mu1>
+      <mu2>10</mu2>
       <fdir1>0 0 0</fdir1>
-      <kp>1e+13</kp>
+      <kp>1e+20</kp>
       <kd>1.0</kd>
       <selfCollide>0</selfCollide>
-      <maxContacts>10</maxContacts>
+      <maxContacts>1</maxContacts>
       <material>Gazebo/Blue</material> <!-- caution this overrwrites (dae) everything!!! -->
    </gazebo>

File: ball_description/urdf/ball.urdf.xacro (robot description, xacro)
@@ -2,4 +2,5 @@
 <robot xmlns:controller="http://playerstage.sourceforge.net/gazebo/xmlschema/#controller" xmlns:interface="http://ros.org/wiki/xacro" xmlns:sensor="http://playerstage.sourceforge.net/gazebo/xmlschema/#sensor" xmlns:xacro="http://ros.org/wiki/xacro" name="$(arg ball_name)">
    <xacro:include filename="$(find ball_description)/urdf/ball.gazebo.xacro" />
+   <xacro:property name="scale_size" value="0.5" />
    <xacro:macro name="ball_macro" params="prefix">
       <link name="${prefix}ball_link">
@@ -7,5 +8,5 @@
          <origin rpy="0 0 0" xyz="0 0 0" />
          <geometry>
-            <mesh filename="package://ball_description/models/tennis_ball/meshes/tennis_ball.dae" scale="1 1 1" />
+            <mesh filename="package://ball_description/models/tennis_ball/meshes/tennis_ball.dae" scale="${scale_size*1} ${scale_size*1} ${scale_size*1}" />
          </geometry>
          <cast_shadows>1</cast_shadows>
@@ -15,11 +16,11 @@
          <inertial>
             <origin xyz="0 0 0" rpy="0 0 0" />
-            <mass value="0.056" />
-            <inertia ixx="0.000038" ixy="0" ixz="0" iyy="0.000038" iyz="0" izz="0.000038" />
+            <mass value="${scale_size*0.056}" />
+            <inertia ixx="${scale_size*0.000038}" ixy="0" ixz="0" iyy="${scale_size*0.000038}" iyz="0" izz="${scale_size*0.000038}" />
          </inertial>
          <collision>
             <origin rpy="0 0 0" xyz="0 0 0" />
             <geometry>
-               <mesh filename="package://ball_description/models/tennis_ball/meshes/tennis_ball.dae" scale="1 1 1" />
+               <mesh filename="package://ball_description/models/tennis_ball/meshes/tennis_ball.dae" scale="${scale_size*1} ${scale_size*1} ${scale_size*1}" />
             </geometry>
          </collision>

File: kr5_description/urdf/kr.gazebo.xacro (robot description, xacro)
@@ -74,4 +74,11 @@
       <gazebo reference="ee_link">
          <material>Gazebo/White</material>
+         <fdir1>0 0 0</fdir1>
+         <kp>1e+13</kp>
+         <kd>1.0</kd>
+         <selfCollide>0</selfCollide>
+         <maxContacts>10</maxContacts>
+         <mu1>10</mu1>
+         <mu2>10</mu2>
       </gazebo>
     </xacro:if>

File: kr5_description/urdf/kr5.urdf.xacro (robot description, xacro)
@@ -173,5 +173,5 @@
            <origin xyz="0 0 0" rpy="0 0 0" />
            <geometry>
-              <mesh filename="package://kr5_description/meshes/tools/plate_40.stl" scale="0.02 0.02 0.02" /> <!-- plate is 20x20x1cm if scale is 0.01 -->
+              <mesh filename="package://kr5_description/meshes/tools/plate_40.stl" scale="0.01 0.01 0.01" /> <!-- plate is 20x20x1cm if scale is 0.01 -->
            </geometry>
         </visual>
@@ -179,5 +179,5 @@
            <origin xyz="0 0 0" rpy="0 0 0" />
            <geometry>
-              <mesh filename="package://kr5_description/meshes/tools/plate_40.stl" scale="0.02 0.02 0.02" /> <!-- plate is 20x20x1 m -->
+              <mesh filename="package://kr5_description/meshes/tools/plate_40.stl" scale="0.01 0.01 0.01" /> <!-- plate is 20x20x1 m -->
            </geometry>
         </collision>
@@ -214,5 +214,5 @@
          <origin xyz="0 -0.12 0" rpy="0 ${-pi/2} 0" />
       <axis xyz="0 0 1" />
-      <limit lower="${radians(-350)}" upper="${radians(350)}" effort="28.0" velocity="3.2"/>
+      <limit lower="${radians(-350)}" upper="${radians(350)}" effort="60.0" velocity="3.2"/> <!-- max should be 28 -->
       <dynamics damping="0.0" friction="0.0"/>
     </joint>
@@ -222,5 +222,5 @@
          <origin xyz="0 0 -0.62" rpy="0 ${pi/2} 0" />
       <axis xyz="0 0 1" />
-      <limit  lower="${radians(-130)}" upper="${radians(130)}" effort="28.0" velocity="3.2"/>
+      <limit  lower="${radians(-130)}" upper="${radians(130)}" effort="60.0" velocity="3.2"/> <!-- max should be 28 -->
       <dynamics damping="0.0" friction="0.0"/>
     </joint>
